File: Model_T_RAM_type_b.kicad_sch (KiCad schematic)
At the start: 5 parts, among them J1 KC-85_RAM, U1 6264, U2 74HC86

Commit message: add type b variant
Parts:
- removed C2: 0.1u, 000_LOCAL:C_0805, symbol 000_LOCAL:C
Connections:
- net A11: now also U2.1; no longer U2.5
- net CE2: now also U2.3; no longer U2.6
- net ~{CS_C}: now also U2.5; no longer U2.2
- net ~{CS_D}: now also U2.4; no longer U2.1
- new net: U2.2, U2.6
Other:
- moved on the sheet: U2A, U2B, U2C, U2D
