File: Model_T_RAM.kicad_sch (KiCad schematic)
At the start: 5 parts, among them J1 KC-85_RAM, U1 6264, U2 74HC86

Commit message: kicad 7
Connections:
- no-connect marks 1 -> 0
Other:
- note added: "VCC is "VB", and has power at all times, whether main power is on or off. RAM_RST goes high before main power transitions, on or off, and stays high while main power is off. RAM_RST protects ram from random writes during power-on & power-off transitions, and keeps ram powered-down while main power is off."
- note removed: "VB"
- note removed: "VCC is "VB", and has power at all times. RAM_RST is high while machine is on standby."
- moved on the sheet: C1, C2, J1, U2A, U2B, U2C, U2D, U2E
